Commit message: tom: 6-DOF wrist, grounded base, 10 mm clamp spacers + URDF/SRDF
Drop the wrist servo (7->6 DOF), ground the base so the clamp underside sits at z=0, regenerate the 10 mm clamp spacers, attach the gripper to the u-bracket, and match the URDF/SRDF default pose to the STEP. Remove the tom_double / tom_with_gripper variants and stale printable samples.

Co-Authored-By: Claude Opus 4.8 <noreply@anthropic.com>

File: models/robots/tom/tom.urdf (robot description, URDF)
Before this commit: robot tom_v2, 9 links, 8 joints
Links:
- removed link wrist_roll_link
- added link gripper_base_link, mass 0.158659843; collision mesh filename=3MF/gripper_static.3mf scale=0.001 0.001 0.001; visual mesh filename=3MF/gripper_static.3mf scale=0.001 0.001 0.001
- added link gripper_left_claw_link, mass 0.044399027; collision mesh filename=3MF/gripper_left_claw.3mf scale=0.001 0.001 0.001; visual mesh filename=3MF/gripper_left_claw.3mf scale=0.001 0.001 0.001
- added link gripper_right_claw_link, mass 0.044399027; collision mesh filename=3MF/gripper_right_claw.3mf scale=0.001 0.001 0.001; visual mesh filename=3MF/gripper_right_claw.3mf scale=0.001 0.001 0.001
- added link gripper_servo_link, mass 0.002542102; collision mesh filename=3MF/gripper_servo_gear.3mf scale=0.001 0.001 0.001; visual mesh filename=3MF/gripper_servo_gear.3mf scale=0.001 0.001 0.001
- link base_link: mass 0.163725567 -> 0.164049472
- link elbow_roll_link: mass 0.151640174 -> 0.1462769; geometry visual mesh filename=3MF/link_bracket_left.3mf scale=0.001 0.001 0.001; visual mesh filename=3MF/link_bracket_right.3mf scale=0.001 0.001 0.001
- link shoulder_roll_link: mass 0.190640174 -> 0.1852769; geometry visual mesh filename=3MF/link_bracket_left.3mf scale=0.001 0.001 0.001; visual mesh filename=3MF/link_bracket_right.3mf scale=0.001 0.001 0.001
Joints:
- removed joint wrist_roll
- added joint gripper_left_claw_slide: type prismatic, parent gripper_base_link, child gripper_left_claw_link, origin xyz=0 0 0 rpy=0 0 0, axis 1 0 0, limit lower=0 upper=0.038000 effort=150 velocity=0.03, mimic joint=gripper_servo multiplier=0.006499998870 offset=0
- added joint gripper_right_claw_slide: type prismatic, parent gripper_base_link, child gripper_right_claw_link, origin xyz=0 0 0 rpy=0 0 0, axis -1 0 0, limit lower=0 upper=0.038000 effort=150 velocity=0.03, mimic joint=gripper_servo multiplier=0.006499998870 offset=0
- added joint gripper_servo: type revolute, parent gripper_base_link, child gripper_servo_link, origin xyz=0 0 0 rpy=0 0 0, axis 0 0 1, limit lower=0 upper=5.846154862 effort=2.941995 velocity=4.615385
- added joint wrist_pitch_to_gripper_base: type fixed, parent wrist_pitch_link, child gripper_base_link, origin xyz=-0.000002072 -0.000033863 -0.0785 rpy=-3.141592512 0 1.571173117
- joint base_footprint_to_base_link: origin xyz=0.014635742 0 0.072518 rpy=1.570796327 0 0 -> xyz=0.014635742 0 0.009343 rpy=1.570796327 0 0
- joint elbow_pitch: origin xyz=0 0 0.1665 rpy=3.141592654 0 1.570796327 -> xyz=0 0 0.1665 rpy=0 -1.570796327 -1.570796327
